File: PCB/Stimulator/Multi Chromatic Stimulator.kicad_pcb (KiCad board)
At the start: 2 copper layers, 125 x 75 mm, 38 parts, among them J2 5V - 30V

Commit message: 2019.05.23
Parts:
- added 2N5089: , Package_TO_SOT_THT:TO-92L_Inline_Wide, F.Cu at (110.8, 64.5)
- added ?: 1k, Maxime:R_Axial_DIN0309_L9.0mm_D3.2mm_P15.24mm_Horizontal, F.Cu at (106.5, 65.3)
- added ?: 1k, Maxime:R_Axial_DIN0309_L9.0mm_D3.2mm_P15.24mm_Horizontal, F.Cu at (106.7, 70.6)
- added ?: PinHeader_1x03_P2.54mm_Vertical, Connector_PinHeader_2.54mm:PinHeader_1x03_P2.54mm_Vertical, F.Cu at (90.7, 65.1)
- J2: value 5V - 30V -> Conn_01x02_Female
- R3: renamed from ?; value 470 Ω -> 470
- R4: renamed from ?; value 220 Ω -> 220
Connections:
- ? pad 3V3: (no net) -> Net-(A1-Pad16)
- J2 pad 1: Net-(J25-Pad1) -> Net-(J2-Pad1)
- J2 pad 2: GNDREF -> Net-(J1-Pad2)
- J2 pad 3: GNDREF -> (no net)
- R3 pad 1: Net-(A1-Pad23) -> GNDREF
- R3 pad 2: GNDREF -> Net-(A2-Pad20)
- R4 pad 1: Net-(A1-Pad23) -> Net-(A2-Pad20)
- R4 pad 2: Net-(A1-Pad23) -> Net-(A1-Pad12)
Routing:
- net Net-(A1-Pad16): track 0.00 -> 55.4 mm
- net Net-(A1-Pad23): track 175.1 -> 190.2 mm
- net Net-(Q1-Pad2): track 0.00 -> 8.77 mm
Other:
- board text added: "2019.05.22"
- board text added: "Multi-Chromatic Stimulator v2.1"
- board text added: "Signal Inverter"
- board text removed: "2018.12.12"
- board text removed: "Multi-Chromatic Stimulator v2.0"

Commit message: Version 2.1 update
Parts:
- added ?: , Connector_PinHeader_2.54mm:PinHeader_1x03_P2.54mm_Vertical, F.Cu at (95.8, 103.2)
- ?: value PinHeader_1x03_P2.54mm_Vertical -> (none)
- J2: value Conn_01x02_Female -> 5V - 30V
- moved ? 2.42 mm to (78.8, 114.2)
- moved ? 2.42 mm to (90.1, 110.7)
- renumbered R3 to ?, R4 to ?
Connections:
- ? pad 1: GNDREF -> Net-(A1-Pad23)
- ? pad 2: Net-(A2-Pad20) -> GNDREF
- ? pad 2: Net-(A1-Pad12) -> Net-(A1-Pad23)
- J2 pad 2: Net-(J1-Pad2) -> GNDREF
- J2 pad 3: (no net) -> GNDREF
Routing:
- net Net-(A1-Pad23): track 190.2 -> 200.7 mm
- net Net-(A2-Pad20): track 0.00 -> 6.75 mm
- net Net-(J25-Pad1): track 875.6 -> 879.9 mm
